File: pcb/TP_Alejandro_Gorrin/TP_Alejandro_Gorrin.sch (KiCad schematic (older format))
At the start: 33 parts, among them J1 Conn_01x12, J2 Conn_01x02, J3 Conn_01x16, Q1 MMBT3904, Q2 MMBT3904, Q3 BS250, SW1 SW_1, U1 MCP73831-2-OT, U2 TPD4S014, U3 CP2104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

Commit message: cambio de nombre al compilar
Parts:
- removed CHG: ORANGE, symbol Device:LED
- added D1: LED, symbol Device:LED
Connections:
- no-connect marks 23 -> 25
Changed lines of the file:
@@
 	0    -1   -1   0
 $EndComp
-$Comp
-L Device:LED CHG
-U 1 1 5F80BE22
-P 1150 5750
-F 0 "CHG" H 1150 5550 50  0000 C CNN
-F 1 "ORANGE" H 1200 5650 50  0000 C CNN
-F 2 "" H 1150 5750 50  0001 C CNN
-F 3 "~" H 1150 5750 50  0001 C CNN
-	1    1150 5750
-	-1   0    0    1
-$EndComp
 Wire Wire Line
 	2150 5750 1750 5750
 Wire Wire Line
 	1450 5750 1300 5750
-Wire Wire Line
-	1000 5750 900  5750
-Wire Wire Line
-	900  5750 900  5600
 Wire Wire Line
 	2150 6900 2150 7000
@@
 	1950 5950 1950 6100
 Wire Wire Line
-	900  6500 900  5750
-Connection ~ 900  5750
-Wire Wire Line
 	2175 1725 2175 1875
 Wire Wire Line
@@
 	1625 1775 1625 1675
 Wire Wire Line
-	1875 1325 1625 1325
-Wire Wire Line
 	1625 1375 1625 1325
 Wire Wire Line
@@
 	1375 1725 1375 1875
 Wire Wire Line
-	725  1475 725  1325
-Wire Wire Line
 	1375 825  1375 725
-Wire Wire Line
-	1075 1025 725  1025
-Connection ~ 725  1025
-Wire Wire Line
-	725  1025 725  725
-Wire Wire Line
-	825  1325 725  1325
-Connection ~ 725  1325
-Wire Wire Line
-	725  1325 725  1025
 Wire Wire Line
 	725  1775 725  1875
@@
 Wire Wire Line
 	1125 1325 1375 1325
-Connection ~ 1625 1325
 Connection ~ 1375 1325
 Wire Wire Line
@@
 NoConn ~ 5225 2150
 NoConn ~ 5225 2350
+$Comp
+L Device:LED D1
+U 1 1 5F85EF33
+P 1150 5750
+F 0 "D1" H 1143 5495 50  0000 C CNN
+F 1 "LED" H 1143 5586 50  0000 C CNN
+F 2 "" H 1150 5750 50  0001 C CNN
+F 3 "~" H 1150 5750 50  0001 C CNN
+	1    1150 5750
+	-1   0    0    1
+$EndComp
+Wire Wire Line
+	1875 1325 1625 1325
+Connection ~ 1625 1325
+NoConn ~ 2125 4850
+NoConn ~ 6250 4600
+Wire Wire Line
+	900  6500 900  5750
+Wire Wire Line
+	1000 5750 900  5750
+Connection ~ 900  5750
+Wire Wire Line
+	900  5750 900  5600
+Wire Wire Line
+	725  725  725  1025
+Wire Wire Line
+	825  1325 725  1325
+Connection ~ 725  1325
+Wire Wire Line
+	725  1325 725  1475
+Wire Wire Line
+	1075 1025 725  1025
+Connection ~ 725  1025
+Wire Wire Line
+	725  1025 725  1325
 $EndSCHEMATC

Commit message: cambio de componente
Parts:
- removed U2: TPD4S014, Package_SON:Texas_S-PWSON-N10, symbol Power_Protection:TPD4S014
- added J4: USB_A, symbol Connector:USB_A
Connections:
- no-connect marks 25 -> 21
Changed lines of the file:
@@
-$EndComp
-$Comp
-L Power_Protection:TPD4S014 U2
-U 1 1 5F823F62
-P 5725 2450
-F 0 "U2" H 5725 3017 50  0000 C CNN
-F 1 "TPD4S014" H 5725 2926 50  0000 C CNN
-F 2 "Package_SON:Texas_S-PWSON-N10" H 6625 1950 50  0001 C CNN
-F 3 "http://www.ti.com/lit/ds/symlink/tpd4s014.pdf" H 6825 1750 50  0001 C CNN
-	1    5725 2450
-	-1   0    0    -1
 $EndComp
 $Comp
@@
 L power:GNDD #PWR0112
 U 1 1 5F8A1CC4
-P 5725 3050
-F 0 "#PWR0112" H 5725 2800 50  0001 C CNN
-F 1 "GNDD" H 5729 2895 50  0000 C CNN
-F 2 "" H 5725 3050 50  0001 C CNN
-F 3 "" H 5725 3050 50  0001 C CNN
-	1    5725 3050
-	1    0    0    -1
-$EndComp
-Wire Wire Line
-	5725 2950 5725 3050
+P 5850 3000
+F 0 "#PWR0112" H 5850 2750 50  0001 C CNN
+F 1 "GNDD" H 5854 2845 50  0000 C CNN
+F 2 "" H 5850 3000 50  0001 C CNN
+F 3 "" H 5850 3000 50  0001 C CNN
+	1    5850 3000
+	1    0    0    -1
+$EndComp
 Wire Wire Line
 	5925 1200 6525 1200
@@
 	6525 1200 6525 1350
 Wire Wire Line
-	6225 2150 6325 2150
-Wire Wire Line
-	6325 2150 6325 1550
-Wire Wire Line
 	6325 1550 6775 1550
 Wire Wire Line
-	6225 2650 6425 2650
-Wire Wire Line
-	6425 2650 6425 1850
-Wire Wire Line
 	6425 1850 6775 1850
 Wire Wire Line
-	6225 2750 6525 2750
-Wire Wire Line
-	6525 2750 6525 1950
-Wire Wire Line
-	6525 1950 6775 1950
-Wire Wire Line
 	6325 1550 6325 1500
-Connection ~ 6325 1550
 Wire Wire Line
 	8175 1550 8375 1550
@@
 NoConn ~ 7575 2950
 NoConn ~ 7475 2950
-NoConn ~ 6225 2350
-NoConn ~ 6225 2550
-NoConn ~ 5625 2950
-NoConn ~ 5225 2150
-NoConn ~ 5225 2350
 $Comp
 L Device:LED D1
@@
 Wire Wire Line
 	725  1025 725  1325
+Connection ~ 6325 1550
+$Comp
+L Connector:USB_A J4
+U 1 1 5F8DC6D3
+P 5850 2450
+F 0 "J4" H 5907 2917 50  0000 C CNN
+F 1 "USB_A" H 5907 2826 50  0000 C CNN
+F 2 "" H 6000 2400 50  0001 C CNN
+F 3 " ~" H 6000 2400 50  0001 C CNN
+	1    5850 2450
+	1    0    0    -1
+$EndComp
+Wire Wire Line
+	5850 2850 5850 3000
+Wire Wire Line
+	6150 2250 6325 2250
+Wire Wire Line
+	6325 1550 6325 2250
+Wire Wire Line
+	6425 2550 6150 2550
+Wire Wire Line
+	6425 1850 6425 2550
+Wire Wire Line
+	6500 1950 6500 2450
+Wire Wire Line
+	6500 2450 6150 2450
+Wire Wire Line
+	6500 1950 6775 1950
+NoConn ~ 5750 2850
 $EndSCHEMATC

Commit message: asignacion de footprint
Parts:
- C1, J4: footprint (none) -> Connector_USB:USB_A_CONNFLY_DS1095-WNR0
- C2, C3, C4, C6, C7, C8: footprint (none) -> Capacitor_SMD:CP_Elec_3x5.3
- D1, D3, D4: footprint (none) -> LED_SMD:LED_0603_1608Metric
- J2: footprint (none) -> Connector_PinHeader_2.54mm:PinHeader_1x02_P2.54mm_Vertical
- R1, R10, R12, R13, R13G1, R13G2, R2, R3, R4, R7: footprint (none) -> Resistor_SMD:R_0201_0603Metric
- SW1: footprint (none) -> Button_Switch_SMD:SW_DIP_SPSTx01_Slide_6.7x4.1mm_W6.73mm_P2.54mm_LowProfile_JPin
Other:
- moved on the sheet: C4, R13, SW1A
Changed lines of the file:
@@
 F 0 "R1" V 2350 7000 50  0000 C CNN
 F 1 "4.7K" V 2450 7000 50  0000 C CNN
-F 2 "" V 2380 7000 50  0001 C CNN
+F 2 "Resistor_SMD:R_0201_0603Metric" V 2380 7000 50  0001 C CNN
 F 3 "~" H 2450 7000 50  0001 C CNN
 	1    2450 7000
@@
 F 0 "R2" V 1500 5700 50  0000 L CNN
 F 1 "1K" V 1600 5700 50  0000 L CNN
-F 2 "" V 1530 5750 50  0001 C CNN
+F 2 "Resistor_SMD:R_0201_0603Metric" V 1530 5750 50  0001 C CNN
 F 3 "~" H 1600 5750 50  0001 C CNN
 	1    1600 5750
@@
 F 0 "C3" H 1550 6100 50  0000 L CNN
 F 1 "10uF" H 1550 6200 50  0000 L CNN
-F 2 "" H 1488 6000 50  0001 C CNN
+F 2 "Capacitor_SMD:CP_Elec_3x5.3" H 1488 6000 50  0001 C CNN
 F 3 "~" H 1450 6150 50  0001 C CNN
 	1    1450 6150
@@
 F 0 "R10" H 3825 6075 50  0000 L CNN
 F 1 "1K" V 3775 6025 50  0000 L CNN
-F 2 "" V 3705 6075 50  0001 C CNN
+F 2 "Resistor_SMD:R_0201_0603Metric" V 3705 6075 50  0001 C CNN
 F 3 "~" H 3775 6075 50  0001 C CNN
 	1    3775 6075
@@
 F 0 "D3" V 3825 6625 50  0000 L CNN
 F 1 "RED" V 3725 6625 50  0000 L CNN
-F 2 "" H 3775 6525 50  0001 C CNN
+F 2 "LED_SMD:LED_0603_1608Metric" H 3775 6525 50  0001 C CNN
 F 3 "~" H 3775 6525 50  0001 C CNN
 	1    3775 6525
@@
 F 0 "D4" H 975 1108 50  0000 C CNN
 F 1 "MBR120" H 975 1199 50  0000 C CNN
-F 2 "" H 975 1325 50  0001 C CNN
+F 2 "LED_SMD:LED_0603_1608Metric" H 975 1325 50  0001 C CNN
 F 3 "~" H 975 1325 50  0001 C CNN
 	1    975  1325
@@
 F 0 "R12" H 795 1671 50  0000 L CNN
 F 1 "100K" V 725 1525 50  0000 L CNN
-F 2 "" V 655 1625 50  0001 C CNN
+F 2 "Resistor_SMD:R_0201_0603Metric" V 655 1625 50  0001 C CNN
 F 3 "~" H 725 1625 50  0001 C CNN
 	1    725  1625
@@
 F 0 "C6" H 1125 1625 50  0000 L CNN
 F 1 "10uF" H 1075 1525 50  0000 L CNN
-F 2 "" H 1413 1425 50  0001 C CNN
+F 2 "Capacitor_SMD:CP_Elec_3x5.3" H 1413 1425 50  0001 C CNN
 F 3 "~" H 1375 1575 50  0001 C CNN
 	1    1375 1575
@@
 F 0 "R7" H 1675 1525 50  0000 L CNN
 F 1 "100K" V 1625 1425 50  0000 L CNN
-F 2 "" V 1555 1525 50  0001 C CNN
+F 2 "Resistor_SMD:R_0201_0603Metric" V 1555 1525 50  0001 C CNN
 F 3 "~" H 1625 1525 50  0001 C CNN
 	1    1625 1525
@@
 F 0 "C7" H 2425 1525 50  0000 L CNN
 F 1 "10uF" H 2425 1425 50  0000 L CNN
-F 2 "" H 2663 1375 50  0001 C CNN
+F 2 "Capacitor_SMD:CP_Elec_3x5.3" H 2663 1375 50  0001 C CNN
 F 3 "~" H 2625 1525 50  0001 C CNN
 	1    2625 1525
@@
 F 0 "C8" H 2775 1525 50  0000 L CNN
 F 1 "10uF" H 2775 1425 50  0000 L CNN
-F 2 "" H 3013 1375 50  0001 C CNN
+F 2 "Capacitor_SMD:CP_Elec_3x5.3" H 3013 1375 50  0001 C CNN
 F 3 "~" H 2975 1525 50  0001 C CNN
 	1    2975 1525
@@
 F 0 "C1" H 3875 1675 50  0000 L CNN
 F 1 "10uF" H 3825 1475 50  0000 L CNN
-F 2 "" H 3863 1425 50  0001 C CNN
+F 2 "Connector_USB:USB_A_CONNFLY_DS1095-WNR0" H 3863 1425 50  0001 C CNN
 F 3 "~" H 3825 1575 50  0001 C CNN
 	1    3825 1575
@@
 L Device:R R13
 U 1 1 5F81E48A
-P 4325 1375
-F 0 "R13" H 4425 1425 50  0000 L CNN
-F 1 "10K" V 4325 1325 50  0000 L CNN
-F 2 "" V 4255 1375 50  0001 C CNN
-F 3 "~" H 4325 1375 50  0001 C CNN
-	1    4325 1375
+P 4325 1275
+F 0 "R13" H 4425 1325 50  0000 L CNN
+F 1 "10K" V 4325 1225 50  0000 L CNN
+F 2 "Resistor_SMD:R_0201_0603Metric" V 4255 1275 50  0001 C CNN
+F 3 "~" H 4325 1275 50  0001 C CNN
+	1    4325 1275
 	1    0    0    -1
 $EndComp
@@
 L Device:C C4
 U 1 1 5F81EACA
-P 4875 1425
-F 0 "C4" H 4675 1425 50  0000 L CNN
-F 1 "1uF" H 4725 1325 50  0000 L CNN
-F 2 "" H 4913 1275 50  0001 C CNN
-F 3 "~" H 4875 1425 50  0001 C CNN
-	1    4875 1425
+P 4875 1325
+F 0 "C4" H 4675 1325 50  0000 L CNN
+F 1 "1uF" H 4725 1225 50  0000 L CNN
+F 2 "Capacitor_SMD:CP_Elec_3x5.3" H 4913 1175 50  0001 C CNN
+F 3 "~" H 4875 1325 50  0001 C CNN
+	1    4875 1325
 	1    0    0    -1
 $EndComp
@@
 F 0 "C2" H 5725 1400 50  0000 L CNN
 F 1 "10uF" H 5725 1300 50  0000 L CNN
-F 2 "" H 5963 1250 50  0001 C CNN
+F 2 "Capacitor_SMD:CP_Elec_3x5.3" H 5963 1250 50  0001 C CNN
 F 3 "~" H 5925 1400 50  0001 C CNN
 	1    5925 1400
@@
 F 0 "R3" H 4075 2900 50  0000 L CNN
 F 1 "100K" V 4225 2750 50  0000 L CNN
-F 2 "" V 4155 2850 50  0001 C CNN
+F 2 "Resistor_SMD:R_0201_0603Metric" V 4155 2850 50  0001 C CNN
 F 3 "~" H 4225 2850 50  0001 C CNN
 	1    4225 2850
@@
 F 0 "R4" H 4075 3400 50  0000 L CNN
 F 1 "100K" V 4225 3250 50  0000 L CNN
-F 2 "" V 4155 3350 50  0001 C CNN
+F 2 "Resistor_SMD:R_0201_0603Metric" V 4155 3350 50  0001 C CNN
 F 3 "~" H 4225 3350 50  0001 C CNN
 	1    4225 3350
@@
 F 0 "R13G1" V 3925 4300 50  0000 C CNN
 F 1 "10K" V 4025 4300 50  0000 C CNN
-F 2 "" V 3955 4300 50  0001 C CNN
+F 2 "Resistor_SMD:R_0201_0603Metric" V 3955 4300 50  0001 C CNN
 F 3 "~" H 4025 4300 50  0001 C CNN
 	1    4025 4300
@@
 F 0 "R13G2" V 4525 4800 50  0000 C CNN
 F 1 "10K" V 4425 4800 50  0000 C CNN
-F 2 "" V 4355 4800 50  0001 C CNN
+F 2 "Resistor_SMD:R_0201_0603Metric" V 4355 4800 50  0001 C CNN
 F 3 "~" H 4425 4800 50  0001 C CNN
 	1    4425 4800
@@
 $EndComp
 Wire Wire Line
-	4875 1575 4875 1825
-Wire Wire Line
-	4875 1275 4875 1075
-Wire Wire Line
-	4325 1525 4325 1575
-Wire Wire Line
-	4325 1225 4325 1125
+	4875 1475 4875 1725
+Wire Wire Line
+	4875 1175 4875 975
+Wire Wire Line
+	4325 1425 4325 1475
+Wire Wire Line
+	4325 1125 4325 1025
 $Comp
 L power:GNDD #PWR0110
 U 1 1 5F87E65D
-P 4875 1825
-F 0 "#PWR0110" H 4875 1575 50  0001 C CNN
-F 1 "GNDD" H 4879 1670 50  0000 C CNN
-F 2 "" H 4875 1825 50  0001 C CNN
-F 3 "" H 4875 1825 50  0001 C CNN
-	1    4875 1825
+P 4875 1725
+F 0 "#PWR0110" H 4875 1475 50  0001 C CNN
+F 1 "GNDD" H 4879 1570 50  0000 C CNN
+F 2 "" H 4875 1725 50  0001 C CNN
+F 3 "" H 4875 1725 50  0001 C CNN
+	1    4875 1725
 	1    0    0    -1
 $EndComp
@@
 L power:+3.3V #PWR0128
 U 1 1 5F8B58CC
-P 4325 1125
-F 0 "#PWR0128" H 4325 975 50  0001 C CNN
-F 1 "+3.3V" H 4340 1298 50  0000 C CNN
-F 2 "" H 4325 1125 50  0001 C CNN
-F 3 "" H 4325 1125 50  0001 C CNN
-	1    4325 1125
+P 4325 1025
+F 0 "#PWR0128" H 4325 875 50  0001 C CNN
+F 1 "+3.3V" H 4340 1198 50  0000 C CNN
+F 2 "" H 4325 1025 50  0001 C CNN
+F 3 "" H 4325 1025 50  0001 C CNN
+	1    4325 1025
 	1    0    0    -1
 $EndComp
@@
 Wire Wire Line
 	3775 5000 3775 5100
-Text Label 4875 1075 0    47   ~ 0
+Text Label 4875 975  0    47   ~ 0
 RESET
 Text Label 725  3450 0    47   ~ 0
@@
 L Switch:SW_DPST_x2 SW1
 U 1 1 5FACBEA5
-P 4325 1825
-F 0 "SW1" V 4375 1775 50  0000 R CNN
-F 1 "SW_1" V 4275 1775 50  0000 R CNN
-F 2 "" H 4325 1825 50  0001 C CNN
-F 3 "~" H 4325 1825 50  0001 C CNN
-	1    4325 1825
+P 4325 1725
+F 0 "SW1" V 4375 1675 50  0000 R CNN
+F 1 "SW_1" V 4275 1675 50  0000 R CNN
+F 2 "Button_Switch_SMD:SW_DIP_SPSTx01_Slide_6.7x4.1mm_W6.73mm_P2.54mm_LowProfile_JPin" H 4325 1725 50  0001 C CNN
+F 3 "~" H 4325 1725 50  0001 C CNN
+	1    4325 1725
 	0    -1   -1   0
 $EndComp
 Wire Wire Line
-	4325 2025 4325 2075
+	4325 1925 4325 1975
 $Comp
 L power:GNDD #PWR0132
 U 1 1 5FAD39A9
-P 4325 2075
-F 0 "#PWR0132" H 4325 1825 50  0001 C CNN
-F 1 "GNDD" H 4325 1950 50  0000 C CNN
-F 2 "" H 4325 2075 50  0001 C CNN
-F 3 "" H 4325 2075 50  0001 C CNN
-	1    4325 2075
-	1    0    0    -1
-$EndComp
-Wire Wire Line
-	4325 1575 4375 1575
-Connection ~ 4325 1575
-Wire Wire Line
-	4325 1575 4325 1625
-Text Label 4375 1575 0    47   ~ 0
+P 4325 1975
+F 0 "#PWR0132" H 4325 1725 50  0001 C CNN
+F 1 "GNDD" H 4325 1850 50  0000 C CNN
+F 2 "" H 4325 1975 50  0001 C CNN
+F 3 "" H 4325 1975 50  0001 C CNN
+	1    4325 1975
+	1    0    0    -1
+$EndComp
+Wire Wire Line
+	4325 1475 4375 1475
+Connection ~ 4325 1475
+Wire Wire Line
+	4325 1475 4325 1525
+Text Label 4375 1475 0    47   ~ 0
 RESET
-$Comp
-L Connector_Generic:Conn_01x02 J2
-U 1 1 5FAE0C0D
-P 3475 1575
-F 0 "J2" H 3425 1675 50  0000 L CNN
-F 1 "Conn_01x02" H 3275 1375 50  0000 L CNN
-F 2 "" H 3475 1575 50  0001 C CNN
-F 3 "~" H 3475 1575 50  0001 C CNN
-	1    3475 1575
-	1    0    0    -1
-$EndComp
 Wire Wire Line
 	3275 1575 3225 1575
@@
 F 0 "D1" H 1143 5495 50  0000 C CNN
 F 1 "LED" H 1143 5586 50  0000 C CNN
-F 2 "" H 1150 5750 50  0001 C CNN
+F 2 "LED_SMD:LED_0603_1608Metric" H 1150 5750 50  0001 C CNN
 F 3 "~" H 1150 5750 50  0001 C CNN
 	1    1150 5750
@@
 F 0 "J4" H 5907 2917 50  0000 C CNN
 F 1 "USB_A" H 5907 2826 50  0000 C CNN
-F 2 "" H 6000 2400 50  0001 C CNN
+F 2 "Connector_USB:USB_A_CONNFLY_DS1095-WNR0" H 6000 2400 50  0001 C CNN
 F 3 " ~" H 6000 2400 50  0001 C CNN
 	1    5850 2450
@@
 	6500 1950 6775 1950
 NoConn ~ 5750 2850
+$Comp
+L Connector_Generic:Conn_01x02 J2
+U 1 1 5F951B62
+P 3475 1575
+F 0 "J2" H 3425 1675 50  0000 L CNN
+F 1 "Conn_01x02" H 3275 1375 50  0000 L CNN
+F 2 "Connector_PinHeader_2.54mm:PinHeader_1x02_P2.54mm_Vertical" H 3475 1575 50  0001 C CNN
+F 3 "~" H 3475 1575 50  0001 C CNN
+	1    3475 1575
+	1    0    0    -1
+$EndComp
 $EndSCHEMATC

Commit message: Agrego PWR FLAGS
Changed lines of the file:
@@
 	1450 5950 1950 5950
 Wire Wire Line
-	1450 6300 1450 6350
-Wire Wire Line
 	1950 5950 1950 6100
 Wire Wire Line
@@
 Wire Wire Line
 	1375 1425 1375 1325
-Wire Wire Line
-	1375 1725 1375 1875
-Wire Wire Line
-	1375 825  1375 725
 Wire Wire Line
 	725  1775 725  1875
@@
 	3775 6225 3775 6375
 Wire Wire Line
-	3775 5925 3775 5775
+	3775 5925 3775 5850
 $Comp
 L Transistor_FET:BS250 Q3
@@
 	3275 1575 3225 1575
 Wire Wire Line
-	3225 1575 3225 1325
-Wire Wire Line
 	3275 1675 3225 1675
-Wire Wire Line
-	3225 1675 3225 1825
 $Comp
 L power:GNDD #PWR0133
 U 1 1 5FAF1249
-P 3225 1825
-F 0 "#PWR0133" H 3225 1575 50  0001 C CNN
-F 1 "GNDD" H 3229 1670 50  0000 C CNN
-F 2 "" H 3225 1825 50  0001 C CNN
-F 3 "" H 3225 1825 50  0001 C CNN
-	1    3225 1825
+P 3225 2000
+F 0 "#PWR0133" H 3225 1750 50  0001 C CNN
+F 1 "GNDD" H 3229 1845 50  0000 C CNN
+F 2 "" H 3225 2000 50  0001 C CNN
+F 3 "" H 3225 2000 50  0001 C CNN
+	1    3225 2000
 	1    0    0    -1
 $EndComp
@@
 $EndComp
 Wire Wire Line
-	1875 1325 1625 1325
+	1875 1325 1750 1325
 Connection ~ 1625 1325
 NoConn ~ 2125 4850
@@
 $EndComp
 Wire Wire Line
-	5850 2850 5850 3000
+	5850 2850 5850 2925
 Wire Wire Line
 	6150 2250 6325 2250
 Wire Wire Line
-	6325 1550 6325 2250
+	6325 1550 6325 1875
 Wire Wire Line
 	6425 2550 6150 2550
@@
 	1    0    0    -1
 $EndComp
+Wire Wire Line
+	1450 6300 1450 6350
+$Comp
+L power:PWR_FLAG #FLG0103
+U 1 1 5F8B58E7
+P 6225 1875
+F 0 "#FLG0103" H 6225 1950 50  0001 C CNN
+F 1 "PWR_FLAG" V 6225 2025 50  0000 L CNN
+F 2 "" H 6225 1875 50  0001 C CNN
+F 3 "~" H 6225 1875 50  0001 C CNN
+	1    6225 1875
+	0    -1   -1   0
+$EndComp
+Wire Wire Line
+	6225 1875 6325 1875
+Connection ~ 6325 1875
+Wire Wire Line
+	6325 1875 6325 2250
+$Comp
+L power:PWR_FLAG #FLG0104
+U 1 1 5F8BEAF5
+P 5975 2925
+F 0 "#FLG0104" H 5975 3000 50  0001 C CNN
+F 1 "PWR_FLAG" V 5975 3053 50  0000 L CNN
+F 2 "" H 5975 2925 50  0001 C CNN
+F 3 "~" H 5975 2925 50  0001 C CNN
+	1    5975 2925
+	0    1    1    0
+$EndComp
+Wire Wire Line
+	5975 2925 5850 2925
+Connection ~ 5850 2925
+Wire Wire Line
+	5850 2925 5850 3000
+$Comp
+L power:PWR_FLAG #FLG0105
+U 1 1 5F8C7B1A
+P 3850 5850
+F 0 "#FLG0105" H 3850 5925 50  0001 C CNN
+F 1 "PWR_FLAG" V 3950 5900 50  0000 L CNN
+F 2 "" H 3850 5850 50  0001 C CNN
+F 3 "~" H 3850 5850 50  0001 C CNN
+	1    3850 5850
+	0    1    1    0
+$EndComp
+Wire Wire Line
+	3850 5850 3775 5850
+Connection ~ 3775 5850
+Wire Wire Line
+	3775 5850 3775 5775
+Wire Wire Line
+	3225 1675 3225 2000
+Wire Wire Line
+	3225 1325 3225 1575
+Wire Wire Line
+	1375 725  1375 825
+Wire Wire Line
+	1375 1725 1375 1875
+$Comp
+L power:PWR_FLAG #FLG0101
+U 1 1 5F8EC339
+P 1750 1300
+F 0 "#FLG0101" H 1750 1375 50  0001 C CNN
+F 1 "PWR_FLAG" H 1675 1450 50  0000 C CNN
+F 2 "" H 1750 1300 50  0001 C CNN
+F 3 "~" H 1750 1300 50  0001 C CNN
+	1    1750 1300
+	1    0    0    -1
+$EndComp
+Wire Wire Line
+	1750 1300 1750 1325
+Connection ~ 1750 1325
+Wire Wire Line
+	1750 1325 1625 1325
 $EndSCHEMATC

Commit message: footprint y componente ESP32
Parts:
- U5: footprint ESP32-footprints-Lib:ESP-32S -> ESP32-footprints-Lib:ESP32
Changed lines of the file:
@@
 F 0 "U5" H 2000 5187 60  0000 C CNN
 F 1 "ESP3212" H 2000 5081 60  0000 C CNN
-F 2 "ESP32-footprints-Lib:ESP-32S" H 2375 5150 60  0001 C CNN
+F 2 "ESP32-footprints-Lib:ESP32" H 2375 5150 60  0001 C CNN
 F 3 "" H 1575 4250 60  0001 C CNN
 	1    2025 3800

Commit message: Cambios del Esquematico
Parts:
- removed U5: ESP3212, ESP32-footprints-Lib:ESP32, symbol ESP32-footprints-Shem-Lib:ESP3212
- added U5: ESP32-WROOM, ESP32-footprints-Lib:ESP32-WROOM, symbol ESP32-footprints-Shem-Lib:ESP32-WROOM
- C1: footprint Connector_USB:USB_A_CONNFLY_DS1095-WNR0 -> Capacitor_SMD:C_0805_2012Metric
- C2, C3, C4, C6, C7, C8: footprint Capacitor_SMD:CP_Elec_3x5.3 -> Capacitor_SMD:C_0805_2012Metric
- D1, D3, D4: footprint LED_SMD:LED_0603_1608Metric -> LED_SMD:LED_0805_2012Metric
- R1, R10, R12, R13, R13G1, R13G2, R2, R3, R4, R7: footprint Resistor_SMD:R_0201_0603Metric -> Resistor_SMD:R_0805_2012Metric
- SW1: footprint Button_Switch_SMD:SW_DIP_SPSTx01_Slide_6.7x4.1mm_W6.73mm_P2.54mm_LowProfile_JPin -> Button_Switch_SMD:SW_Push_1P1T_NO_6x6mm_H9.5mm
Connections:
- net +3V3: now also U5.2 (3V3)
- net A0_DAC2: now also U5.11 (IO26)
- net A13_I35: now also U5.7 (IO35)
- net A1_DAC1: now also U5.10 (IO25)
- net A2_I34: now also U5.6 (IO34)
- net A3_I39: now also U5.5 (SENSOR_VN)
- net A4_IO36: now also U5.4 (SENSOR_VP)
- net A5_IO4: now also U5.26 (IO4)
- net GNDD: now also R1.2, U5.1 (GND), U5.15 (GND); no longer R1.1
- net GPIO0: now also U5.25 (IO0)
- net GPIO2: now also U5.24 (IO2)
- net IO12_A11: now also U5.14 (IO12)
- net IO13_A12: now also U5.16 (IO13)
- net IO14_A6: now also U5.13 (IO14)
- net IO15_A8: now also U5.23 (IO15)
- net IO16: now also U5.27 (IO16)
- net IO17: now also U5.28 (IO17)
- net IO21: now also U5.33 (IO21)
- net IO27_A10: now also U5.12 (IO27)
- net IO32_A7: now also U5.8 (IO32)
- net IO33_A9: now also U5.9 (IO33)
- net MISI: now also U5.30 (IO18)
- net MISO: now also U5.31 (IO19)
- net RESET: now also U5.3 (EN)
- net RXD0: now also U5.34 (RXD0)
- net SCI: now also U5.36 (IO22)
- net SCK: now also U5.29 (IO5)
- net SDA: now also U5.37 (IO23)
- net TXD0: now also U5.35 (TXD0)
- net at U1.5 (PROG): now also R1.1; no longer R1.2
- no-connect marks 21 -> 27
Other:
- moved on the sheet: C3, C4, D1, R1, R13, R2, SW1A, U1

Commit message: Agrego avances de PCB, problemas con el heatsink
Connections:
- net IO13_A1 is gone; now on net IO13_A12: R10.2
Changed lines of the file:
@@
 RESET
 Text Label 3775 5775 0    47   ~ 0
-IO13_A1
+IO13_A12
 Wire Wire Line
 	2975 1175 2975 1325

Commit message: Avances PCB
Parts:
- removed HS1: Heatsink_Pad, Heatsink:Heatsink_35x26mm_1xFixation3mm_Fischer-SK486-35, symbol Mechanical:Heatsink_Pad
- removed J4: USB_A, Connector_USB:USB_A_CONNFLY_DS1095-WNR0, symbol Connector:USB_A
- added J4: USB_B_Micro, Connector_USB:USB_Micro-B_Molex_47346-0001, symbol Connector:USB_B_Micro
Connections:
- net GNDD: now also J4.5 (GND)
- net VBUS: now also J4.1 (VBUS)
- net at U3.3 (D+): now also J4.3 (D+)
- net at U3.4 (D-): now also J4.2 (D-)
- no-connect marks 27 -> 28
Changed lines of the file:
@@
 Wire Wire Line
 	1375 1225 1375 1325
-$Comp
-L Mechanical:Heatsink_Pad HS1
-U 1 1 5F941341
-P 6675 3250
-F 0 "HS1" H 6816 3289 50  0000 L CNN
-F 1 "Heatsink_Pad" H 6816 3198 50  0000 L CNN
-F 2 "Heatsink:Heatsink_35x26mm_1xFixation3mm_Fischer-SK486-35" H 6687 3200 50  0001 C CNN
-F 3 "~" H 6687 3200 50  0001 C CNN
-	1    6675 3250
-	1    0    0    -1
-$EndComp
-Wire Wire Line
-	6675 3350 6675 3450
-$Comp
-L power:GNDD #PWR0131
-U 1 1 5F945A4A
-P 6675 3450
-F 0 "#PWR0131" H 6675 3200 50  0001 C CNN
-F 1 "GNDD" H 6679 3295 50  0000 C CNN
-F 2 "" H 6675 3450 50  0001 C CNN
-F 3 "" H 6675 3450 50  0001 C CNN
-	1    6675 3450
-	1    0    0    -1
-$EndComp
 Text Label 8375 1550 0    47   ~ 0
 DTR
@@
 	725  1025 725  1325
 Connection ~ 6325 1550
-$Comp
-L Connector:USB_A J4
-U 1 1 5F8DC6D3
-P 5850 2450
-F 0 "J4" H 5907 2917 50  0000 C CNN
-F 1 "USB_A" H 5907 2826 50  0000 C CNN
-F 2 "Connector_USB:USB_A_CONNFLY_DS1095-WNR0" H 6000 2400 50  0001 C CNN
-F 3 " ~" H 6000 2400 50  0001 C CNN
-	1    5850 2450
-	1    0    0    -1
-$EndComp
 Wire Wire Line
 	6150 2250 6325 2250
@@
 Wire Wire Line
 	2850 6825 2850 6500
+$Comp
+L Connector:USB_B_Micro J4
+U 1 1 5FA8962C
+P 5850 2450
+F 0 "J4" H 5907 2917 50  0000 C CNN
+F 1 "USB_B_Micro" H 5907 2826 50  0000 C CNN
+F 2 "Connector_USB:USB_Micro-B_Molex_47346-0001" H 6000 2400 50  0001 C CNN
+F 3 "~" H 6000 2400 50  0001 C CNN
+	1    5850 2450
+	1    0    0    -1
+$EndComp
+NoConn ~ 6150 2650
 $EndSCHEMATC
