File: pcb/TP_Alejandro_Gorrin/TP_Alejandro_Gorrin.kicad_pcb (KiCad board)
At the start: 2 copper layers, 36 parts, among them J1 Conn_01x12, J2 Conn_01x02, J3 Conn_01x16, J4 USB_B_Micro, Q1 MMBT3904, Q2 MMBT3904, Q3 BS250, SW1 SW_1, U1 MCP73831-2-OT, U3 CP2104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

Commit message: PCB cambios
Parts:
- removed MK103, MK104: MountingHole, MountingHole:MountingHole_2.2mm_M2_DIN965_Pad
- Q3: value BS250 -> DMG3414U; footprint Package_TO_SOT_THT:TO-92_Inline -> Package_TO_SOT_SMD:SOT-23
- moved MK102 3.30 mm to (124.9, 111.0)
- moved MK101 3.14 mm to (125.0, 84.9)
- moved Q3 2.07 mm to (132.4, 94.2), turned to 90 degrees
- moved C2 0.40 mm to (145.4, 100.1)
- moved C3 0.40 mm to (129.1, 85.0)
- moved C4 0.40 mm to (139.9, 97.8)
- moved C6 0.40 mm to (134.5, 90.4)
- moved C7 0.40 mm to (142.6, 92.5)
- moved D3 0.40 mm to (142.9, 100.2)
- moved D4 0.40 mm to (144.4, 88.5)
- moved J1 0.40 mm to (139.8, 84.3)
- moved J2 0.40 mm to (135.0, 84.3)
- moved J3 0.40 mm to (129.6, 111.8)
- moved Q1 0.40 mm to (131.7, 103.9)
- moved Q2 0.40 mm to (129.4, 107.7)
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Connections:
- J4 pad 5: Net-(J4-Pad5) -> GNDD
- Q3 pad 1: +BATT -> VBUS
- Q3 pad 2: VBUS -> +BATT
Routing:
- net GNDD: track 99.2 -> 48.5 mm
- net VBUS: track 47.4 -> 51.2 mm, vias 7 -> 5
- net (no net): track 0.00 -> 3.00 mm
- net Net-(C6-Pad1): track 19.3 -> 16.9 mm, vias 3 -> 2
- net +BATT: track 43.4 -> 42.7 mm
- added copper zone on B.Cu, net GNDD
- added copper zone on F.Cu, net GNDD
Other:
- board outline added: 53 x 32 mm
